File: Schematics/ScreenGrabV2/grab.sch (EAGLE design)
At the start: 48 parts

Commit message: Schematic routed
Parts:
- removed JP5: (no value), pinhead:PINHD-2X24
- removed VCC/GND: (no value), pinhead:PINHD-1X2
- added C29, C30, C31, C32, C33, C34, C35, C36, C39, C42, C43, C44, C45: (no value), resistor:C-EUC0603
- added CN1: 4p-2.54-h8.5, Seeed-OPL-Connector:DIP-SCREW-TERMINAL-GREEN(4P-2.54-H8.5)
- added CN3: 2p-2.54-h8.5, Seeed-OPL-Connector:DIP-SCREW-TERMINAL-GREEN(2P-2.54-H8.5)
- added D1, D6: CLEAR-BLUE-0805, Seeed-OPL-Diode:SMD-LED-CLEAR-BLUE(0805)
- added D2, D3, D4, D5: BLUE-0603, Seeed-OPL-Diode:SMD-LED-CLEAR-BLUE(0603)
- added J2: MICROSD-9P, Seeed-OPL-Connector:MICRO-SD-CARD-HOLDER-9P
- added JP1: (no value), pinhead:PINHD-2X3
- added JP2: (no value), pinhead:PINHD-2X25
- added R10, R11, R12, R13, R14, R5: (no value), resistor:R-EU_R0603
- added U3, U5: ATMEGA328P-AU-TQFP32, Seeed-OPL-ic:MCU-ATMEGA328P-AU(TQFP32)
- added U4, U6: (no value), SparkFun-PowerIC:V_REG_LM1117SOT223
- added Y1, Y2: 16MHZ, Seeed-OPL-crystal-osctllator:SMD-CRYSTAL-16MHZ-8PF-20PPM-40R(2P-5.0X3.2MM)
- JP3: device pinhead:PINHD-1X4 -> pinhead:PINHD-2X3
- JP4: device pinhead:PINHD-2X15 -> pinhead:PINHD-2X25
- JP6: device pinhead:PINHD-2X15 -> pinhead:PINHD-2X3
Connections:
- new net C_MISO: JP6.1, U5.PB4(MISO)
- new net C_MOSI: JP6.4, U5.PB3(MOSI/OC2)
- new net C_RST: JP6.5, U5.PC6(/RESET)
- new net C_SCK: JP6.3, R5.2, U5.PB5(SCK)
- new net C_VCC: C42.1, C44.1, C45.1, JP6.2, U5.AREF, U5.AVCC, U5.VCC@1, U5.VCC@2, U6.OUT, U6.OUT@1
- new net N$10: C30.1, U3.PB6(XTAL1/TOSC1), Y1.1
- new net N$11: C29.1, U3.PB7(XTAL2/TOSC2), Y1.2
- new net N$12: D2.-, R10.1
- new net N$13: D3.-, R11.1
- new net N$14: D4.-, R12.1
- new net N$15: D5.-, R13.1
- new net N$16: D6.+, U5.ADC7
- new net N$17: D6.-, R14.1
- new net N$2: J2.CS, U3.PB2(SS/OC1B)
- new net N$3: D2.+, U3.PD5(T1)
- new net N$4: C39.1, U5.PB6(XTAL1/TOSC1), Y2.1
- new net N$5: C36.1, U5.PB7(XTAL2/TOSC2), Y2.2
- new net N$6: D3.+, U3.PD6(AIN0)
- new net N$7: D4.+, U3.PD7(AIN1)
- new net N$8: D1.+, R5.1
- new net N$9: D5.+, U3.PB0(ICP)
- new net UNUSED1: JP4.17, U3.PD0(RXD)
- new net UNUSED2: JP4.15, U3.PD1(TXD)
- new net UNUSED3: JP4.13, U3.PD2(INT0)
- new net W_MISO: J2.DO, JP1.1, U3.PB4(MISO)
- new net W_MOSI: J2.DI, JP1.4, U3.PB3(MOSI/OC2)
- new net W_RST: JP1.5, U3.PC6(/RESET)
- new net W_SCK: J2.SCLK, JP1.3, U3.PB5(SCK)
- new net W_VCC: C31.1, C32.1, C34.1, C35.1, J2.VDD, JP1.2, U3.AREF, U3.AVCC, U3.VCC@1, U3.VCC@2, U4.OUT, U4.OUT@1
- net +3.3V: now also JP3.4
- net +5V: now also C33.1, C43.1, CN3.2, U4.IN, U6.IN; no longer VCC/GND.2
- net B0: now also JP2.14; no longer JP4.14
- net B1: now also JP2.13; no longer JP4.13
- net B2: now also JP2.12; no longer JP4.12
- net B3: now also JP2.11; no longer JP4.11
- net B4: now also JP2.10; no longer JP4.10
- net B5: now also JP2.9; no longer JP4.9
- net B6: now also JP2.8; no longer JP4.8
- net B7: now also JP2.7; no longer JP4.7
- net BIN: now also CN1.3; no longer JP3.3
- net CSYNCIN: now also CN1.4; no longer JP3.4
- net FIDOUT: now also JP4.11; no longer JP6.14
- net G0: now also JP2.22; no longer JP4.22
- net G1: now also JP2.21; no longer JP4.21
- net G2: now also JP2.20; no longer JP4.20
- net G3: now also JP2.19; no longer JP4.19
- net G4: now also JP2.18; no longer JP4.18
- net G5: now also JP2.17; no longer JP4.17
- net G6: now also JP2.16; no longer JP4.16
- net G7: now also JP2.15; no longer JP4.15
- net GIN: now also CN1.2; no longer JP3.2
- net GND: now also C29.2, C30.2, C31.2, C32.2, C33.2, C34.2, C35.2, C36.2, C39.2, C42.2, C43.2, C44.2, C45.2, CN3.1, D1.-, J2.G1, J2.G2, J2.G3, J2.G4, J2.VSS, JP1.6, JP2.2, JP2.4, JP3.5, JP3.6, JP6.6, R10.2, R11.2, R13.2, R14.2, U3.GND, U3.GND@1, U3.GND@2, U4.ADJ, U5.GND, U5.GND@1, U5.GND@2, U6.ADJ; no longer JP4.2, JP4.4, VCC/GND.1
- net HSOUT: now also JP4.7; no longer JP6.10
- net N$1: now also JP2.1; no longer JP4.1
- net PCLK: now also JP4.5; no longer JP6.8
- net R0: now also JP2.30; no longer JP4.30
- net R1: now also JP2.29; no longer JP4.29
- net R2: now also JP2.28; no longer JP4.28
- net R3: now also JP2.27; no longer JP4.27
- net R4: now also JP2.26; no longer JP4.26
- net R5: now also JP2.25; no longer JP4.25
- net R6: now also JP2.24; no longer JP4.24
- net R7: now also JP2.23; no longer JP4.23
- net RESET: now also JP3.3, U5.PB2(SS/OC1B)
- net RIN: now also CN1.1; no longer JP3.1
- net SCL: now also JP3.2, U5.PC5(ADC5/SCL)
- net SDA: now also JP3.1, U5.PC4(ADC4/SDA)
- net VSOUT: now also JP4.9; no longer JP6.12

Commit message: Schematic update
Parts:
- added GRAB: 2p-2.54-h8.5, Seeed-OPL-Connector:DIP-SCREW-TERMINAL-GREEN(2P-2.54-H8.5)
- added R15: 10K, resistor:R-EU_R0603
- VREG1, VREG3, VREG4: value (none) -> 3.3V
- VREG2: value (none) -> 1.8V
- renumbered CN3 to VCC/GND, D1 to DONE, D2 to LED1, D3 to LED2, D4 to LED3, D5 to LED4, D6 to LED5, JP1 to ISP_OUT, JP3 to I2C, JP6 to ISP_CTRL, U1 to VREG1, U2 to VREG2, U3 to MEGA328_OUT, U4 to VREG4, U5 to MEGA328_CTRL, U6 to VREG3
Connections:
- removed net UNUSED3: JP4.13, MEGA328_OUT.PD2(INT0)
- new net CAPTURE: GRAB.1, JP4.13, MEGA328_OUT.PD2(INT0), R15.2
- net +3.3V: now also R15.1
- net GND: now also GRAB.2
